Commit message: Stabilize Gazebo drive physics and simplify RViz

File: ros2_ws/description/robot_core.xacro (robot description, xacro)
@@ -32,5 +32,5 @@
          for four-wheel skid-steer turning. These require real-world tuning. -->
     <xacro:property name="tire_ground_mu_longitudinal" value="0.85"/>
-    <xacro:property name="tire_ground_mu_lateral" value="0.45"/>
+    <xacro:property name="tire_ground_mu_lateral" value="0.12"/>
     <!--
       MGL42GM-895, 24 V, 71:1 gearbox (the purchased 140 RPM version).
@@ -150,5 +150,5 @@
                             y="${chassis_width}"
                             z="${chassis_height}">
-            <origin xyz="0 0 0" rpy="0 0 0"/>
+            <origin xyz="-0.080 0 -0.050" rpy="0 0 0"/>
         </xacro:inertial_box>
     </link>
@@ -349,7 +349,7 @@
             </visual>
             <collision>
-                <origin xyz="0 0 0" rpy="${pi / 2} 0 0"/>
-                <geometry>
-                    <cylinder radius="${wheel_radius}" length="${wheel_width}"/>
+                <origin xyz="0 0 0" rpy="0 0 0"/>
+                <geometry>
+                    <sphere radius="${wheel_radius}"/>
                 </geometry>
             </collision>
