Commit message: Feat: Expand forklift simulation and manual controls

File: ros2_ws/description/forklift.xacro (robot description, xacro)
@@ -21,4 +21,24 @@
     <!-- At lift_joint=0, the underside of each fork is 65 mm above ground. -->
     <xacro:property name="fork_ground_clearance" value="0.065"/>
+    <!--
+      Lift drivetrain, synchronized with ESP32 Projects/cang_nang_ha:
+      - 1.8 degree stepper, >=0.7 N.m holding torque
+      - direct-drive T8x8 lead screw (8 mm travel per revolution)
+      - 50 mm/s maximum travel = 375 screw RPM
+      The supplied stepper sheet has no torque-speed curve. At 375 RPM, use a
+      conservative 50% of holding torque and 30% T8 screw efficiency. This
+      gives about 82.47 N available axial lift force. Update these two factors
+      after measuring current and lift force on the real mechanism.
+    -->
+    <xacro:property name="stepper_holding_torque" value="0.700"/>
+    <xacro:property name="stepper_running_torque_factor" value="0.50"/>
+    <xacro:property name="t8_screw_lead" value="0.008"/>
+    <xacro:property name="t8_screw_efficiency" value="0.30"/>
+    <xacro:property name="lift_max_velocity" value="0.05"/>
+    <xacro:property name="stepper_available_torque"
+                    value="${stepper_holding_torque * stepper_running_torque_factor}"/>
+    <xacro:property name="lift_max_force"
+                    value="${2.0 * pi * t8_screw_efficiency
+                             * stepper_available_torque / t8_screw_lead}"/>
     <!-- Dimensions below are visual estimates pending direct measurement. -->
     <xacro:property name="mast_profile" value="0.030"/>
@@ -185,5 +205,6 @@
                     rpy="0 0 0"/>
             <axis xyz="0 0 1"/>
-            <limit lower="0.0" upper="${lift_travel}" effort="1000.0" velocity="0.05"/>
+            <limit lower="0.0" upper="${lift_travel}"
+                   effort="${lift_max_force}" velocity="${lift_max_velocity}"/>
             <dynamics damping="5.0" friction="2.0"/>
         </joint>

File: ros2_ws/description/gazebo_control.xacro (robot description, xacro)
@@ -37,12 +37,16 @@
             <initial_position>0.0</initial_position>
             <p_gain>1200.0</p_gain>
-            <i_gain>20.0</i_gain>
+            <!-- Feed-forward already balances gravity; integral action caused
+                 about 14 mm of wind-up after a long upward move. -->
+            <i_gain>0.0</i_gain>
             <d_gain>80.0</d_gain>
             <i_min>-100.0</i_min>
             <i_max>100.0</i_max>
-            <cmd_min>-1000.0</cmd_min>
-            <cmd_max>1000.0</cmd_max>
+            <!-- Prismatic joint commands are force [N], limited by the
+                 estimated stepper + T8x8 drivetrain capability. -->
+            <cmd_min>${-lift_max_force}</cmd_min>
+            <cmd_max>${lift_max_force}</cmd_max>
             <!-- Feed-forward balances the estimated 4 kg moving assembly. -->
-            <cmd_offset>39.24</cmd_offset>
+            <cmd_offset>${moving_fork_mass * 9.81}</cmd_offset>
         </plugin>
         <!-- Gazebo joint feedback is bridged to ROS /joint_states. -->

File: ros2_ws/description/imu_bno055.xacro (robot description, xacro)
@@ -109,4 +109,25 @@
             </xacro:inertial_box>
         </link>
+        <!-- Gazebo Harmonic IMU. Axes follow imu_link / REP-103. -->
+        <gazebo reference="imu_link">
+            <sensor name="imu_sensor" type="imu">
+                <always_on>true</always_on>
+                <update_rate>100</update_rate>
+                <topic>/imu</topic>
+                <gz_frame_id>imu_link</gz_frame_id>
+                <imu>
+                    <angular_velocity>
+                        <x><noise type="gaussian"><mean>0</mean><stddev>0.0002</stddev></noise></x>
+                        <y><noise type="gaussian"><mean>0</mean><stddev>0.0002</stddev></noise></y>
+                        <z><noise type="gaussian"><mean>0</mean><stddev>0.0002</stddev></noise></z>
+                    </angular_velocity>
+                    <linear_acceleration>
+                        <x><noise type="gaussian"><mean>0</mean><stddev>0.017</stddev></noise></x>
+                        <y><noise type="gaussian"><mean>0</mean><stddev>0.017</stddev></noise></y>
+                        <z><noise type="gaussian"><mean>0</mean><stddev>0.017</stddev></noise></z>
+                    </linear_acceleration>
+                </imu>
+            </sensor>
+        </gazebo>
     </xacro:macro>
 </robot>

File: ros2_ws/description/robot_core.xacro (robot description, xacro)
@@ -4,4 +4,5 @@
     <xacro:include filename="forklift.xacro"/>
     <xacro:include filename="imu_bno055.xacro"/>
+    <xacro:include filename="lidar.xacro"/>
     <xacro:include filename="gazebo_control.xacro"/>
     <xacro:include filename="battery_pack.xacro"/>
@@ -24,5 +25,22 @@
     <xacro:property name="tire_ground_mu_longitudinal" value="0.85"/>
     <xacro:property name="tire_ground_mu_lateral" value="0.45"/>
-    <!-- MGL42GM-895, 24 V / 100 RPM (100:1 gearbox), from the supplied drawing. -->
+    <!--
+      MGL42GM-895, 24 V, 71:1 gearbox (the purchased 140 RPM version).
+      Datasheet column 71: 140 RPM no-load, 126 RPM rated,
+      30 kgf.cm rated torque and 98 kgf.cm stall torque.
+      wheel_joint effort uses stall torque as the short-duration peak needed
+      to start a skid-steer turn. The rated torque remains the continuous
+      thermal limit; Gazebo does not model motor temperature or duty cycle.
+    -->
+    <xacro:property name="motor_gear_ratio" value="71.0"/>
+    <xacro:property name="motor_no_load_speed_rpm" value="140.0"/>
+    <xacro:property name="motor_rated_speed_rpm" value="126.0"/>
+    <xacro:property name="kgf_cm_to_nm" value="0.0980665"/>
+    <xacro:property name="motor_rated_torque"
+                    value="${30.0 * kgf_cm_to_nm}"/>
+    <xacro:property name="motor_stall_torque"
+                    value="${98.0 * kgf_cm_to_nm}"/>
+    <xacro:property name="motor_no_load_speed_rad_s"
+                    value="${motor_no_load_speed_rpm * 2.0 * pi / 60.0}"/>
     <xacro:property name="motor_body_length" value="0.072"/>
     <xacro:property name="motor_body_radius" value="0.025"/>
@@ -236,4 +254,7 @@
             <origin xyz="${x} ${y} 0" rpy="0 0 0"/>
             <axis xyz="0 1 0"/>
+            <!-- 9.611 N.m short-duration peak; continuous rating is 2.942 N.m. -->
+            <limit effort="${motor_stall_torque}"
+                   velocity="${motor_no_load_speed_rad_s}"/>
             <dynamics damping="0.1" friction="0.1"/>
         </joint>
@@ -357,4 +378,6 @@
     <!-- Front lift mast and the 0-520 mm prismatic fork mechanism. -->
     <xacro:forklift_assembly parent="base_link"/>
+    <!-- Fixed 360-degree lidar; its scan plane is 0.80 m above the ground. -->
+    <xacro:fork_mast_lidar parent="mast_frame"/>
     <!-- BNO055 mounted near the centre of the chassis top surface. -->
     <xacro:bno055_imu parent="chassis" x="0.0" y="0.0" yaw="0.0"/>

Commit message: Back up current robot project with checked reverse recovery
Snapshot matches community workspace commit 660f5c8. Preserve existing backup history; exclude generated build, install, and log directories.

File: ros2_ws/description/forklift.xacro (robot description, xacro)
@@ -19,6 +19,30 @@
                     value="${fork_gap / 2 + fork_width / 2}"/>
     <xacro:property name="lift_travel" value="0.520"/>
+    <!-- One millimetre of numerical margin prevents Gazebo's physical stop
+         and tiny negative round-off from fighting the PID target at 0.000 m.
+         Public commands and real hardware remain 0.000-0.520 m. -->
+    <xacro:property name="lift_joint_limit_margin" value="0.001"/>
     <!-- At lift_joint=0, the underside of each fork is 65 mm above ground. -->
     <xacro:property name="fork_ground_clearance" value="0.065"/>
+    <!--
+      Lift drivetrain, synchronized with ESP32 Projects/cang_nang_ha:
+      - 1.8 degree stepper, >=0.7 N.m holding torque
+      - direct-drive T8x8 lead screw (8 mm travel per revolution)
+      - 50 mm/s maximum travel = 375 screw RPM
+      The supplied stepper sheet has no torque-speed curve. At 375 RPM, use a
+      conservative 50% of holding torque and 30% T8 screw efficiency. This
+      gives about 82.47 N available axial lift force. Update these two factors
+      after measuring current and lift force on the real mechanism.
+    -->
+    <xacro:property name="stepper_holding_torque" value="0.700"/>
+    <xacro:property name="stepper_running_torque_factor" value="0.50"/>
+    <xacro:property name="t8_screw_lead" value="0.008"/>
+    <xacro:property name="t8_screw_efficiency" value="0.30"/>
+    <xacro:property name="lift_max_velocity" value="0.05"/>
+    <xacro:property name="stepper_available_torque"
+                    value="${stepper_holding_torque * stepper_running_torque_factor}"/>
+    <xacro:property name="lift_max_force"
+                    value="${2.0 * pi * t8_screw_efficiency
+                             * stepper_available_torque / t8_screw_lead}"/>
     <!-- Dimensions below are visual estimates pending direct measurement. -->
     <xacro:property name="mast_profile" value="0.030"/>
@@ -185,5 +209,7 @@
                     rpy="0 0 0"/>
             <axis xyz="0 0 1"/>
-            <limit lower="0.0" upper="${lift_travel}" effort="1000.0" velocity="0.05"/>
+            <limit lower="${-lift_joint_limit_margin}"
+                   upper="${lift_travel + lift_joint_limit_margin}"
+                   effort="${lift_max_force}" velocity="${lift_max_velocity}"/>
             <dynamics damping="5.0" friction="2.0"/>
         </joint>

File: ros2_ws/description/gazebo_control.xacro (robot description, xacro)
@@ -1,55 +1,18 @@
 <?xml version="1.0"?>
 <robot xmlns:xacro="http://www.ros.org/wiki/xacro">
-    <!-- Gazebo Harmonic native controllers for the four-wheel skid-steer base. -->
-    <xacro:macro name="gazebo_control_plugins">
-      <gazebo>
-        <plugin filename="gz-sim-diff-drive-system"
-                name="gz::sim::systems::DiffDrive">
-            <left_joint>front_left_wheel_joint</left_joint>
-            <left_joint>rear_left_wheel_joint</left_joint>
-            <right_joint>front_right_wheel_joint</right_joint>
-            <right_joint>rear_right_wheel_joint</right_joint>
-            <wheel_separation>${wheel_track}</wheel_separation>
-            <wheel_radius>${wheel_radius}</wheel_radius>
-            <odom_publish_frequency>50</odom_publish_frequency>
-            <topic>/cmd_vel</topic>
-            <odom_topic>/odom</odom_topic>
-            <tf_topic>/tf</tf_topic>
-            <frame_id>odom</frame_id>
-            <child_frame_id>base_footprint</child_frame_id>
-            <min_linear_velocity>-0.40</min_linear_velocity>
-            <max_linear_velocity>0.40</max_linear_velocity>
-            <min_angular_velocity>-1.20</min_angular_velocity>
-            <max_angular_velocity>1.20</max_angular_velocity>
-            <min_linear_acceleration>-0.50</min_linear_acceleration>
-            <max_linear_acceleration>0.50</max_linear_acceleration>
-            <min_angular_acceleration>-1.50</min_angular_acceleration>
-            <max_angular_acceleration>1.50</max_angular_acceleration>
-        </plugin>
-        <!--
-          Position target is in metres. The PID drives the carriage while the
-          URDF joint limits enforce the physical 0-0.52 m travel.
-        -->
-        <plugin filename="gz-sim-joint-position-controller-system"
-                name="gz::sim::systems::JointPositionController">
-            <joint_name>lift_joint</joint_name>
-            <topic>/lift_position</topic>
-            <initial_position>0.0</initial_position>
-            <p_gain>1200.0</p_gain>
-            <i_gain>20.0</i_gain>
-            <d_gain>80.0</d_gain>
-            <i_min>-100.0</i_min>
-            <i_max>100.0</i_max>
-            <cmd_min>-1000.0</cmd_min>
-            <cmd_max>1000.0</cmd_max>
-            <!-- Feed-forward balances the estimated 4 kg moving assembly. -->
-            <cmd_offset>39.24</cmd_offset>
-        </plugin>
-        <!-- Gazebo joint feedback is bridged to ROS /joint_states. -->
-        <plugin filename="gz-sim-joint-state-publisher-system"
-                name="gz::sim::systems::JointStatePublisher">
-            <topic>/joint_states</topic>
-        </plugin>
-      </gazebo>
+    <!--
+      Gazebo owns the simulated hardware only.  Drive kinematics, odometry,
+      joint feedback and lift commands are all handled by ros2_control.
+    -->
+    <xacro:macro name="gazebo_ros2_control_plugin" params="controllers_file">
+        <gazebo>
+            <plugin filename="libgz_ros2_control-system.so"
+                    name="gz_ros2_control::GazeboSimROS2ControlPlugin">
+                <parameters>${controllers_file}</parameters>
+                <controller_manager_name>controller_manager</controller_manager_name>
+                <hold_joints>true</hold_joints>
+                <position_proportional_gain>0.1</position_proportional_gain>
+            </plugin>
+        </gazebo>
     </xacro:macro>
 </robot>

File: ros2_ws/description/robot_core.xacro (robot description, xacro)
@@ -4,4 +4,8 @@
     <xacro:include filename="forklift.xacro"/>
     <xacro:include filename="imu_bno055.xacro"/>
+    <xacro:include filename="lidar.xacro"/>
+    <xacro:include filename="camera_astra_pro.xacro"/>
+    <xacro:include filename="sensor_mount.xacro"/>
+    <xacro:include filename="ros2_control.xacro"/>
     <xacro:include filename="gazebo_control.xacro"/>
     <xacro:include filename="battery_pack.xacro"/>
@@ -16,4 +20,9 @@
     <xacro:property name="wheel_radius" value="0.0875"/>
     <xacro:property name="wheel_width" value="0.035"/>
+    <!-- Safety limit used by both the body controller and each wheel command
+         interface.  0.50 m/s corresponds to 5.714 rad/s at this radius. -->
+    <xacro:property name="max_vehicle_linear_speed" value="0.50"/>
+    <xacro:property name="max_wheel_speed_rad_s"
+                    value="${max_vehicle_linear_speed / wheel_radius}"/>
     <!-- Estimated total mass of one rubber-tyred, plastic-rim wheel. -->
     <xacro:property name="wheel_mass" value="0.5"/>
@@ -23,6 +32,23 @@
          for four-wheel skid-steer turning. These require real-world tuning. -->
     <xacro:property name="tire_ground_mu_longitudinal" value="0.85"/>
-    <xacro:property name="tire_ground_mu_lateral" value="0.45"/>
-    <!-- MGL42GM-895, 24 V / 100 RPM (100:1 gearbox), from the supplied drawing. -->
+    <xacro:property name="tire_ground_mu_lateral" value="0.12"/>
+    <!--
+      MGL42GM-895, 24 V, 71:1 gearbox (the purchased 140 RPM version).
+      Datasheet column 71: 140 RPM no-load, 126 RPM rated,
+      30 kgf.cm rated torque and 98 kgf.cm stall torque.
+      wheel_joint effort uses stall torque as the short-duration peak needed
+      to start a skid-steer turn. The rated torque remains the continuous
+      thermal limit; Gazebo does not model motor temperature or duty cycle.
+    -->
+    <xacro:property name="motor_gear_ratio" value="71.0"/>
+    <xacro:property name="motor_no_load_speed_rpm" value="140.0"/>
+    <xacro:property name="motor_rated_speed_rpm" value="126.0"/>
+    <xacro:property name="kgf_cm_to_nm" value="0.0980665"/>
+    <xacro:property name="motor_rated_torque"
+                    value="${30.0 * kgf_cm_to_nm}"/>
+    <xacro:property name="motor_stall_torque"
+                    value="${98.0 * kgf_cm_to_nm}"/>
+    <xacro:property name="motor_no_load_speed_rad_s"
+                    value="${motor_no_load_speed_rpm * 2.0 * pi / 60.0}"/>
     <xacro:property name="motor_body_length" value="0.072"/>
     <xacro:property name="motor_body_radius" value="0.025"/>
@@ -124,5 +150,5 @@
                             y="${chassis_width}"
                             z="${chassis_height}">
-            <origin xyz="0 0 0" rpy="0 0 0"/>
+            <origin xyz="-0.080 0 -0.050" rpy="0 0 0"/>
         </xacro:inertial_box>
     </link>
@@ -236,4 +262,7 @@
             <origin xyz="${x} ${y} 0" rpy="0 0 0"/>
             <axis xyz="0 1 0"/>
+            <!-- 9.611 N.m short-duration peak; continuous rating is 2.942 N.m. -->
+            <limit effort="${motor_stall_torque}"
+                   velocity="${motor_no_load_speed_rad_s}"/>
             <dynamics damping="0.1" friction="0.1"/>
         </joint>
@@ -320,7 +349,7 @@
             </visual>
             <collision>
-                <origin xyz="0 0 0" rpy="${pi / 2} 0 0"/>
-                <geometry>
-                    <cylinder radius="${wheel_radius}" length="${wheel_width}"/>
+                <origin xyz="0 0 0" rpy="0 0 0"/>
+                <geometry>
+                    <sphere radius="${wheel_radius}"/>
                 </geometry>
             </collision>
@@ -357,9 +386,21 @@
     <!-- Front lift mast and the 0-520 mm prismatic fork mechanism. -->
     <xacro:forklift_assembly parent="base_link"/>
+    <!-- Common top bracket: lidar eye at 0.835 m and Astra Pro eye at 0.800 m. -->
+    <xacro:mast_sensor_mount parent="mast_frame"/>
     <!-- BNO055 mounted near the centre of the chassis top surface. -->
     <xacro:bno055_imu parent="chassis" x="0.0" y="0.0" yaw="0.0"/>
     <!-- Rear-mounted 8S2P 32140 LiFePO4 battery inside the chassis. -->
     <xacro:lfp_battery_pack parent="chassis"/>
-    <!-- Native Gazebo Harmonic drive, lift and joint-state systems. -->
-    <xacro:gazebo_control_plugins/>
+    <!-- Stable controller-facing contract shared by simulation and hardware. -->
+    <xacro:tai_robot_ros2_control hardware_plugin="$(arg hardware_plugin)"/>
+    <!-- The Gazebo plugin creates controller_manager inside the simulated
+         model.  A real-hardware launch starts controller_manager itself. -->
+    <xacro:if value="$(arg use_sim)">
+        <xacro:simulated_fork_safety_lidar parent="base_footprint"/>
+        <!-- Simulation rear low scanner; real reverse recovery requires an equivalent sensor. -->
+        <xacro:simulated_fork_safety_lidar parent="base_footprint"
+            prefix="rear" x="-0.34" z="0.12" yaw="${pi}"/>
+        <xacro:gazebo_ros2_control_plugin
+            controllers_file="$(arg controllers_file)"/>
+    </xacro:if>
 </robot>
