Commit message: feat: integrate real robot SLAM sensors and controls

File: ros2_ws/description/forklift.xacro (robot description, xacro)
@@ -26,5 +26,5 @@
     <xacro:property name="fork_ground_clearance" value="0.065"/>
     <!--
-      Lift drivetrain, synchronized with ESP32 Projects/cang_nang_ha:
+      Lift drivetrain, synchronized with ESP32 Projects/bno055_imu_monitor:
       - 1.8 degree stepper, >=0.7 N.m holding torque
       - direct-drive T8x8 lead screw (8 mm travel per revolution)

File: ros2_ws/description/lidar.xacro (robot description, xacro)
@@ -23,5 +23,6 @@
             <origin xyz="${x} ${y} ${z}" rpy="0 0 0"/>
         </joint>
-        <!-- lidar_link is the optical scan plane, exactly z=0.835 m. -->
+        <!-- lidar_link is the optical scan plane. Its absolute height is set
+             by the selected temporary or final mounting joint. -->
         <link name="lidar_link">
             <visual name="a1m8_base_visual">

File: ros2_ws/description/robot.urdf.xacro (robot description, xacro)
@@ -12,4 +12,5 @@
     <xacro:arg name="drive_serial_port" default="/dev/tai_drive"/>
     <xacro:arg name="lift_serial_port" default="/dev/tai_lift"/>
+    <xacro:arg name="use_lift" default="true"/>
     <xacro:arg name="home_lift_on_activate" default="true"/>
     <xacro:arg name="serial_startup_timeout_ms" default="3000"/>

File: ros2_ws/description/robot_core.xacro (robot description, xacro)
@@ -11,5 +11,5 @@
     <xacro:include filename="battery_pack.xacro"/>
     <!-- All dimensions are in metres and all masses are in kilograms. -->
-    <xacro:property name="chassis_length" value="0.605"/>
+    <xacro:property name="chassis_length" value="0.601"/>
     <xacro:property name="chassis_width" value="0.290"/>
     <xacro:property name="chassis_height" value="0.210"/>
@@ -128,5 +128,5 @@
     </joint>
     <link name="base_link"/>
-    <!-- Chassis: 605 x 290 x 210 mm, with its bottom 125 mm above ground. -->
+    <!-- Chassis: 601 x 290 x 210 mm, with its bottom 125 mm above ground. -->
     <joint name="chassis_joint" type="fixed">
         <parent link="base_link"/>
@@ -386,6 +386,18 @@
     <!-- Front lift mast and the 0-520 mm prismatic fork mechanism. -->
     <xacro:forklift_assembly parent="base_link"/>
-    <!-- Common top bracket: lidar eye at 0.835 m and Astra Pro eye at 0.800 m. -->
-    <xacro:mast_sensor_mount parent="mast_frame"/>
+    <!-- Simulation/final bracket keeps both sensors at their designed height.
+         On the current real robot only the camera is on that bracket; the
+         lidar temporarily sits directly on the chassis top. -->
+    <xacro:if value="$(arg use_sim)">
+        <xacro:mast_sensor_mount parent="mast_frame" include_lidar="true"/>
+    </xacro:if>
+    <xacro:unless value="$(arg use_sim)">
+        <xacro:mast_sensor_mount parent="mast_frame" include_lidar="false"/>
+        <!-- Chassis front is +0.3005 m. The scan axis is 0.437 m behind that
+             edge, hence x=-0.1365 m. The A1M8 scan plane is 50 mm above its
+             bottom, which rests on the 0.335 m-high chassis top. -->
+        <xacro:fork_mast_lidar parent="base_footprint"
+                               x="-0.1365" y="0.0" z="0.385"/>
+    </xacro:unless>
     <!-- BNO055 mounted near the centre of the chassis top surface. -->
     <xacro:bno055_imu parent="chassis" x="0.0" y="0.0" yaw="0.0"/>

File: ros2_ws/description/ros2_control.xacro (robot description, xacro)
@@ -15,4 +15,5 @@
                     <param name="lift_serial_port">$(arg lift_serial_port)</param>
                     <param name="lift_baud">115200</param>
+                    <param name="use_lift">$(arg use_lift)</param>
                     <param name="startup_timeout_ms">$(arg serial_startup_timeout_ms)</param>
                     <param name="telemetry_timeout_ms">$(arg serial_telemetry_timeout_ms)</param>
@@ -65,23 +66,33 @@
                 <state_interface name="velocity"/>
             </joint>
-            <!-- Position is metres above the mechanical lower stop. -->
-            <joint name="lift_joint">
-                <xacro:if value="$(arg use_sim)">
+            <!-- Position is metres above the mechanical lower stop. In real
+                 mode with use_lift=false the combined IMU/lift bridge owns
+                 lift_joint and publishes its feedback on /joint_states. -->
+            <xacro:if value="$(arg use_sim)">
+                <joint name="lift_joint">
                     <command_interface name="effort">
                         <param name="min">${-lift_max_force}</param>
                         <param name="max">${lift_max_force}</param>
                     </command_interface>
+                    <state_interface name="position">
+                        <param name="initial_value">0.0</param>
+                    </state_interface>
+                    <state_interface name="velocity"/>
+                </joint>
+            </xacro:if>
+            <xacro:unless value="$(arg use_sim)">
+                <xacro:if value="$(arg use_lift)">
+                    <joint name="lift_joint">
+                        <command_interface name="position">
+                            <param name="min">0.0</param>
+                            <param name="max">${lift_travel}</param>
+                        </command_interface>
+                        <state_interface name="position">
+                            <param name="initial_value">0.0</param>
+                        </state_interface>
+                        <state_interface name="velocity"/>
+                    </joint>
                 </xacro:if>
-                <xacro:unless value="$(arg use_sim)">
-                    <command_interface name="position">
-                        <param name="min">0.0</param>
-                        <param name="max">${lift_travel}</param>
-                    </command_interface>
-                </xacro:unless>
-                <state_interface name="position">
-                    <param name="initial_value">0.0</param>
-                </state_interface>
-                <state_interface name="velocity"/>
-            </joint>
+            </xacro:unless>
         </ros2_control>
     </xacro:macro>

File: ros2_ws/description/sensor_mount.xacro (robot description, xacro)
@@ -49,5 +49,5 @@
         <color rgba="0.85 0.035 0.02 1"/>
     </material>
-    <xacro:macro name="mast_sensor_mount" params="parent">
+    <xacro:macro name="mast_sensor_mount" params="parent include_lidar:=true">
         <!-- The mount frame lies on the laser scan plane. Because the mast is
              fixed, lifting the fork carriage does not move either sensor. -->
@@ -105,6 +105,8 @@
             </xacro:inertial_box>
         </link>
-        <xacro:fork_mast_lidar parent="sensor_mount_link"
-                               x="${lidar_x_on_mount}" y="0" z="0"/>
+        <xacro:if value="${include_lidar}">
+            <xacro:fork_mast_lidar parent="sensor_mount_link"
+                                   x="${lidar_x_on_mount}" y="0" z="0"/>
+        </xacro:if>
         <xacro:astra_pro_camera parent="sensor_mount_link"
                                 x="${camera_x_on_mount}" y="0"
