Commit message: Add Astra Pro camera and sensor mount simulation

File: ros2_ws/description/lidar.xacro (robot description, xacro)
@@ -8,5 +8,6 @@
     <xacro:property name="lidar_turret_radius" value="0.033"/>
     <xacro:property name="lidar_mass" value="0.170"/>
-    <xacro:property name="lidar_scan_height_ground" value="0.800"/>
+    <!-- Measured on the real robot: ground to the centre of the laser eye. -->
+    <xacro:property name="lidar_scan_height_ground" value="0.835"/>
     <material name="lidar_black">
         <color rgba="0.035 0.040 0.045 1"/>
@@ -15,17 +16,16 @@
         <color rgba="0.75 0.04 0.04 1"/>
     </material>
-    <xacro:macro name="fork_mast_lidar" params="parent">
-        <!-- mast_frame starts mast_bottom_ground metres above the floor. -->
+    <xacro:macro name="fork_mast_lidar"
+                 params="parent x:=0.0 y:=0.0 z:=0.0">
         <joint name="lidar_joint" type="fixed">
             <parent link="${parent}"/>
             <child link="lidar_link"/>
-            <origin xyz="${guide_axis_x} 0
-                         ${lidar_scan_height_ground - mast_bottom_ground}"
-                    rpy="0 0 0"/>
+            <origin xyz="${x} ${y} ${z}" rpy="0 0 0"/>
         </joint>
-        <!-- lidar_link is the optical scan plane, exactly z=0.80 m at rest. -->
+        <!-- lidar_link is the optical scan plane, exactly z=0.835 m. -->
         <link name="lidar_link">
             <visual name="a1m8_base_visual">
-                <origin xyz="0 0 -0.0425" rpy="0 0 0"/>
+                <!-- Bottom of the lidar sits on the common sensor plate. -->
+                <origin xyz="0 0 -0.0375" rpy="0 0 0"/>
                 <geometry>
                     <box size="${lidar_body_width} ${lidar_body_depth} 0.025"/>
@@ -34,12 +34,12 @@
             </visual>
             <visual name="a1m8_turret_visual">
-                <origin xyz="0 0 -0.015" rpy="0 0 0"/>
+                <origin xyz="0 0 -0.0125" rpy="0 0 0"/>
                 <geometry>
-                    <cylinder radius="${lidar_turret_radius}" length="0.030"/>
+                    <cylinder radius="${lidar_turret_radius}" length="0.035"/>
                 </geometry>
                 <material name="lidar_red"/>
             </visual>
             <visual name="a1m8_top_cap_visual">
-                <origin xyz="0 0 -0.0025" rpy="0 0 0"/>
+                <origin xyz="0 0 0.0025" rpy="0 0 0"/>
                 <geometry>
                     <cylinder radius="${lidar_turret_radius * 0.72}" length="0.005"/>
@@ -47,13 +47,8 @@
                 <material name="lidar_black"/>
             </visual>
-            <visual name="lidar_bracket_visual">
-                <origin xyz="${-guide_axis_x / 2} 0 -0.045" rpy="0 0 0"/>
-                <geometry>
-                    <box size="${guide_axis_x + 0.010} 0.055 0.010"/>
-                </geometry>
-                <material name="bearing_dark"/>
-            </visual>
             <collision name="a1m8_body_collision">
-                <origin xyz="0 0 ${-lidar_body_height / 2}" rpy="0 0 0"/>
+                <!-- The scan plane is 5 mm below the top of the housing. -->
+                <origin xyz="0 0 ${-lidar_body_height / 2 + 0.005}"
+                        rpy="0 0 0"/>
                 <geometry>
                     <box size="${lidar_body_width} ${lidar_body_depth} ${lidar_body_height}"/>
@@ -64,5 +59,6 @@
                                 y="${lidar_body_depth}"
                                 z="${lidar_body_height}">
-                <origin xyz="0 0 ${-lidar_body_height / 2}" rpy="0 0 0"/>
+                <origin xyz="0 0 ${-lidar_body_height / 2 + 0.005}"
+                        rpy="0 0 0"/>
             </xacro:inertial_box>
         </link>

File: ros2_ws/description/robot_core.xacro (robot description, xacro)
@@ -5,4 +5,6 @@
     <xacro:include filename="imu_bno055.xacro"/>
     <xacro:include filename="lidar.xacro"/>
+    <xacro:include filename="camera_astra_pro.xacro"/>
+    <xacro:include filename="sensor_mount.xacro"/>
     <xacro:include filename="gazebo_control.xacro"/>
     <xacro:include filename="battery_pack.xacro"/>
@@ -378,6 +380,6 @@
     <!-- Front lift mast and the 0-520 mm prismatic fork mechanism. -->
     <xacro:forklift_assembly parent="base_link"/>
-    <!-- Fixed 360-degree lidar; its scan plane is 0.80 m above the ground. -->
-    <xacro:fork_mast_lidar parent="mast_frame"/>
+    <!-- Common top bracket: lidar eye at 0.835 m and Astra Pro eye at 0.800 m. -->
+    <xacro:mast_sensor_mount parent="mast_frame"/>
     <!-- BNO055 mounted near the centre of the chassis top surface. -->
     <xacro:bno055_imu parent="chassis" x="0.0" y="0.0" yaw="0.0"/>

Commit message: feat: unify Nav2 simulation and optimize shortest-route goal handling

File: ros2_ws/description/lidar.xacro (robot description, xacro)
@@ -8,6 +8,12 @@
     <xacro:property name="lidar_turret_radius" value="0.033"/>
     <xacro:property name="lidar_mass" value="0.170"/>
-    <!-- Measured on the real robot: ground to the centre of the laser eye. -->
+    <!-- Designed mast-bracket scan height; the installed real/simulated A1M8
+         currently uses the lower temporary chassis mount below. -->
     <xacro:property name="lidar_scan_height_ground" value="0.835"/>
+    <!-- Validated real-robot lidar extrinsic, shared with Gazebo. -->
+    <xacro:property name="lidar_installed_x" value="-0.2115"/>
+    <xacro:property name="lidar_installed_y" value="0.0"/>
+    <xacro:property name="lidar_installed_z" value="0.385"/>
+    <xacro:property name="lidar_installed_yaw" value="${-2.0 * pi / 180.0}"/>
     <material name="lidar_black">
         <color rgba="0.035 0.040 0.045 1"/>
@@ -74,6 +80,6 @@
                      Express the laser eye pose in that physics link. -->
                 <parent_link>base_footprint</parent_link>
-                <sensor_pose>${chassis_length / 2.0 + mast_profile / 2.0 + lidar_x_on_mount} 0
-                              ${lidar_scan_height_ground} 0 0 0</sensor_pose>
+                <sensor_pose>${lidar_installed_x} ${lidar_installed_y}
+                              ${lidar_installed_z} 0 0 ${lidar_installed_yaw}</sensor_pose>
                 <topic>/scan</topic>
                 <!-- Run the A1M8 at exactly 7 revolutions/second, within its

File: ros2_ws/description/robot_core.xacro (robot description, xacro)
@@ -386,21 +386,19 @@
     <!-- Front lift mast and the 0-520 mm prismatic fork mechanism. -->
     <xacro:forklift_assembly parent="base_link"/>
-    <!-- Simulation/final bracket keeps both sensors at their designed height.
-         On the current real robot only the camera is on that bracket; the
-         lidar temporarily sits directly on the chassis top. -->
+    <!-- Gazebo's camera data use +X forward: a positive URDF Y rotation
+         points +X downward. Keep the existing real-camera calibration until
+         its point-cloud driver can be checked independently. -->
     <xacro:if value="$(arg use_sim)">
-        <xacro:mast_sensor_mount parent="mast_frame" include_lidar="true"/>
+        <xacro:mast_sensor_mount parent="mast_frame" include_lidar="false"
+                                 camera_pitch="${20.0 * pi / 180.0}"/>
     </xacro:if>
     <xacro:unless value="$(arg use_sim)">
-        <!-- The camera on the real bracket is pitched 20 degrees downward. -->
         <xacro:mast_sensor_mount parent="mast_frame" include_lidar="false"
                                  camera_pitch="${-20.0 * pi / 180.0}"/>
-        <!-- Real-robot scan alignment calibration: the temporary lidar mount
-             is 0.2115 m behind base_footprint. The A1M8 scan plane is 50 mm
-             above its bottom, which rests on the 0.335 m-high chassis top. -->
-        <xacro:fork_mast_lidar parent="base_footprint"
-                               x="-0.2115" y="0.0" z="0.385"
-                               yaw="${-2.0 * pi / 180.0}"/>
     </xacro:unless>
+    <!-- Both lidars use the validated temporary chassis mount. -->
+    <xacro:fork_mast_lidar parent="base_footprint"
+                           x="${lidar_installed_x}" y="${lidar_installed_y}"
+                           z="${lidar_installed_z}" yaw="${lidar_installed_yaw}"/>
     <!-- BNO055 mounted near the centre of the chassis top surface. -->
     <xacro:bno055_imu parent="chassis" x="0.0" y="0.0" yaw="0.0"/>

File: ros2_ws/description/sensor_mount.xacro (robot description, xacro)
@@ -10,6 +10,6 @@
     <xacro:property name="sensor_riser_width" value="${mast_profile}"/>
     <xacro:property name="sensor_mount_mass" value="0.200"/>
-    <!-- Both devices stand on the plate. The camera is farther forward (+X)
-         and its eye is 35 mm lower than the lidar scan plane. -->
+    <!-- The camera stands on this plate. Dimensions retain the optional
+         future high-LiDAR bracket; the current LiDAR sits on the chassis. -->
     <xacro:property name="camera_front_overhang" value="0.010"/>
     <!-- sensor_mount_link is on the aluminium-extrusion centreline. This puts
@@ -18,6 +18,6 @@
                     value="${guide_axis_x + shaft_support_depth / 2.0
                              + camera_front_overhang}"/>
-    <!-- Put the lidar behind the camera with a 4 mm physical gap between
-         their housings, while keeping both devices on the same plate. -->
+    <!-- Optional high mount places the lidar behind the camera with a 4 mm
+         physical gap between housings. -->
     <xacro:property name="sensor_housing_gap" value="0.004"/>
     <xacro:property name="lidar_x_on_mount"
@@ -51,6 +51,6 @@
     <xacro:macro name="mast_sensor_mount"
                  params="parent include_lidar:=true camera_pitch:=0.0">
-        <!-- The mount frame lies on the laser scan plane. Because the mast is
-             fixed, lifting the fork carriage does not move either sensor. -->
+        <!-- This mount frame lies at the designed high scan plane. The mast
+             is fixed, so lifting the fork carriage does not move the camera. -->
         <joint name="sensor_mount_joint" type="fixed">
             <parent link="${parent}"/>
