Commit message: Integrate ROS 2 control, navigation, teleop, and ESP32 firmware

File: ros2_ws/description/camera_astra_pro.xacro (robot description, xacro)
@@ -9,6 +9,10 @@
     <xacro:property name="astra_vertical_fov" value="${49.5 * pi / 180.0}"/>
     <xacro:property name="astra_diagonal_fov" value="${73.0 * pi / 180.0}"/>
-    <xacro:property name="astra_image_width" value="640"/>
-    <xacro:property name="astra_image_height" value="480"/>
+    <!-- Laptop-friendly simulation profile. 320 x 240 at 10 Hz preserves the
+         camera geometry while producing 12x fewer pixels per second than
+         640 x 480 at 30 Hz. -->
+    <xacro:property name="astra_image_width" value="320"/>
+    <xacro:property name="astra_image_height" value="240"/>
+    <xacro:property name="astra_update_rate" value="10"/>
     <xacro:property name="astra_fx"
                     value="${(astra_image_width / 2.0)
@@ -17,4 +21,11 @@
                     value="${(astra_image_height / 2.0)
                              / tan(astra_vertical_fov / 2.0)}"/>
+    <!-- Rendering and measurement limits are intentionally different.
+         An object closer than the Astra depth limit still physically occludes
+         the RGB and IR cameras; using 0.6 m as the renderer near plane makes
+         Gazebo incorrectly draw the background through that object.  Render
+         from 5 mm, then astra_sim_range_filter marks measurements below the
+         real 0.6 m limit invalid on the ROS depth and point-cloud topics. -->
+    <xacro:property name="astra_render_near" value="0.005"/>
     <xacro:property name="astra_min_depth" value="0.6"/>
     <xacro:property name="astra_max_depth" value="8.0"/>
@@ -98,12 +109,19 @@
             <sensor name="astra_pro_rgbd" type="rgbd_camera">
                 <always_on>true</always_on>
-                <update_rate>30</update_rate>
+                <update_rate>${astra_update_rate}</update_rate>
                 <visualize>false</visualize>
                 <topic>/camera</topic>
-                <gz_frame_id>camera_link_optical</gz_frame_id>
+                <!-- Gazebo Harmonic generates RGB-D points in its native
+                     camera coordinates: X forward, Y left, Z up. Setting an
+                     optical_frame_id changes only the message header; it does
+                     not rotate the XYZ values into ROS optical coordinates.
+                     Label the simulated data with the frame it actually uses
+                     so TF performs the camera_link -> optical conversion only
+                     when a consumer explicitly requests the optical frame. -->
+                <gz_frame_id>camera_link</gz_frame_id>
                 <camera>
-                    <optical_frame_id>camera_link_optical</optical_frame_id>
+                    <optical_frame_id>camera_link</optical_frame_id>
                     <!-- Separate fx/fy values below reproduce 60 deg horizontal
-                         and 49.5 deg vertical FOV at 640 x 480. -->
+                         and 49.5 deg vertical FOV at the selected resolution. -->
                     <horizontal_fov>${astra_horizontal_fov}</horizontal_fov>
                     <image>
@@ -112,5 +130,5 @@
                     </image>
                     <clip>
-                        <near>${astra_min_depth}</near>
+                        <near>${astra_render_near}</near>
                         <far>${astra_max_depth}</far>
                     </clip>

File: ros2_ws/description/forklift.xacro (robot description, xacro)
@@ -19,4 +19,8 @@
                     value="${fork_gap / 2 + fork_width / 2}"/>
     <xacro:property name="lift_travel" value="0.520"/>
+    <!-- One millimetre of numerical margin prevents Gazebo's physical stop
+         and tiny negative round-off from fighting the PID target at 0.000 m.
+         Public commands and real hardware remain 0.000-0.520 m. -->
+    <xacro:property name="lift_joint_limit_margin" value="0.001"/>
     <!-- At lift_joint=0, the underside of each fork is 65 mm above ground. -->
     <xacro:property name="fork_ground_clearance" value="0.065"/>
@@ -205,5 +209,6 @@
                     rpy="0 0 0"/>
             <axis xyz="0 0 1"/>
-            <limit lower="0.0" upper="${lift_travel}"
+            <limit lower="${-lift_joint_limit_margin}"
+                   upper="${lift_travel + lift_joint_limit_margin}"
                    effort="${lift_max_force}" velocity="${lift_max_velocity}"/>
             <dynamics damping="5.0" friction="2.0"/>

File: ros2_ws/description/gazebo_control.xacro (robot description, xacro)
@@ -1,59 +1,18 @@
 <?xml version="1.0"?>
 <robot xmlns:xacro="http://www.ros.org/wiki/xacro">
-    <!-- Gazebo Harmonic native controllers for the four-wheel skid-steer base. -->
-    <xacro:macro name="gazebo_control_plugins">
-      <gazebo>
-        <plugin filename="gz-sim-diff-drive-system"
-                name="gz::sim::systems::DiffDrive">
-            <left_joint>front_left_wheel_joint</left_joint>
-            <left_joint>rear_left_wheel_joint</left_joint>
-            <right_joint>front_right_wheel_joint</right_joint>
-            <right_joint>rear_right_wheel_joint</right_joint>
-            <wheel_separation>${wheel_track}</wheel_separation>
-            <wheel_radius>${wheel_radius}</wheel_radius>
-            <odom_publish_frequency>50</odom_publish_frequency>
-            <topic>/cmd_vel</topic>
-            <odom_topic>/odom</odom_topic>
-            <tf_topic>/tf</tf_topic>
-            <frame_id>odom</frame_id>
-            <child_frame_id>base_footprint</child_frame_id>
-            <min_linear_velocity>-0.40</min_linear_velocity>
-            <max_linear_velocity>0.40</max_linear_velocity>
-            <min_angular_velocity>-1.20</min_angular_velocity>
-            <max_angular_velocity>1.20</max_angular_velocity>
-            <min_linear_acceleration>-0.50</min_linear_acceleration>
-            <max_linear_acceleration>0.50</max_linear_acceleration>
-            <min_angular_acceleration>-1.50</min_angular_acceleration>
-            <max_angular_acceleration>1.50</max_angular_acceleration>
-        </plugin>
-        <!--
-          Position target is in metres. The PID drives the carriage while the
-          URDF joint limits enforce the physical 0-0.52 m travel.
-        -->
-        <plugin filename="gz-sim-joint-position-controller-system"
-                name="gz::sim::systems::JointPositionController">
-            <joint_name>lift_joint</joint_name>
-            <topic>/lift_position</topic>
-            <initial_position>0.0</initial_position>
-            <p_gain>1200.0</p_gain>
-            <!-- Feed-forward already balances gravity; integral action caused
-                 about 14 mm of wind-up after a long upward move. -->
-            <i_gain>0.0</i_gain>
-            <d_gain>80.0</d_gain>
-            <i_min>-100.0</i_min>
-            <i_max>100.0</i_max>
-            <!-- Prismatic joint commands are force [N], limited by the
-                 estimated stepper + T8x8 drivetrain capability. -->
-            <cmd_min>${-lift_max_force}</cmd_min>
-            <cmd_max>${lift_max_force}</cmd_max>
-            <!-- Feed-forward balances the estimated 4 kg moving assembly. -->
-            <cmd_offset>${moving_fork_mass * 9.81}</cmd_offset>
-        </plugin>
-        <!-- Gazebo joint feedback is bridged to ROS /joint_states. -->
-        <plugin filename="gz-sim-joint-state-publisher-system"
-                name="gz::sim::systems::JointStatePublisher">
-            <topic>/joint_states</topic>
-        </plugin>
-      </gazebo>
+    <!--
+      Gazebo owns the simulated hardware only.  Drive kinematics, odometry,
+      joint feedback and lift commands are all handled by ros2_control.
+    -->
+    <xacro:macro name="gazebo_ros2_control_plugin" params="controllers_file">
+        <gazebo>
+            <plugin filename="libgz_ros2_control-system.so"
+                    name="gz_ros2_control::GazeboSimROS2ControlPlugin">
+                <parameters>${controllers_file}</parameters>
+                <controller_manager_name>controller_manager</controller_manager_name>
+                <hold_joints>true</hold_joints>
+                <position_proportional_gain>0.1</position_proportional_gain>
+            </plugin>
+        </gazebo>
     </xacro:macro>
 </robot>

File: ros2_ws/description/lidar.xacro (robot description, xacro)
@@ -63,37 +63,29 @@
             </xacro:inertial_box>
         </link>
-        <gazebo reference="lidar_link">
-            <sensor name="rplidar_a1m8" type="gpu_lidar">
-                <always_on>true</always_on>
-                <!-- A1M8 nominal rotation rate is 5.5 revolutions/second. -->
-                <update_rate>5.5</update_rate>
-                <!-- RViz still displays /scan; disable the duplicate Gazebo
-                     ray visualization to avoid an extra render workload. -->
-                <visualize>false</visualize>
+        <!-- Gazebo Harmonic's Ogre1 GpuRays backend returns zero for every ray
+             on Ubuntu 24.04.  Use DART physics raycasts so RGB-D may keep the
+             stable Ogre1 renderer while /scan remains independent of graphics. -->
+        <gazebo>
+            <plugin filename="libtai_physics_lidar.so"
+                    name="tai_robot_one::PhysicsLidar">
+                <frame_id>lidar_link</frame_id>
+                <!-- Fixed joints are lumped into base_footprint by URDF->SDF.
+                     Express the laser eye pose in that physics link. -->
+                <parent_link>base_footprint</parent_link>
+                <sensor_pose>${chassis_length / 2.0 + mast_profile / 2.0 + lidar_x_on_mount} 0
+                              ${lidar_scan_height_ground} 0 0 0</sensor_pose>
                 <topic>/scan</topic>
-                <gz_frame_id>lidar_link</gz_frame_id>
-                <ray>
-                    <scan>
-                        <horizontal>
-                            <!-- 360 rays give one-degree angular spacing,
-                                 matching the published A1 angular-resolution limit. -->
-                            <samples>360</samples>
-                            <resolution>1</resolution>
-                            <min_angle>${-pi}</min_angle>
-                            <max_angle>${pi}</max_angle>
-                        </horizontal>
-                    </scan>
-                    <range>
-                        <min>0.15</min>
-                        <max>12.0</max>
-                        <resolution>0.01</resolution>
-                    </range>
-                    <noise>
-                        <type>gaussian</type>
-                        <mean>0</mean>
-                        <stddev>0.003</stddev>
-                    </noise>
-                </ray>
-            </sensor>
+                <!-- Run the A1M8 at exactly 7 revolutions/second, within its
+                     manufacturer-supported configurable scan-rate range. -->
+                <update_rate>7.0</update_rate>
+                <!-- Preserve the A1M8 sampling rate of approximately 8 kHz:
+                     1143 samples/rev * 7 rev/s = 8001 samples/s. -->
+                <samples>1143</samples>
+                <angle_min>${-pi}</angle_min>
+                <angle_max>${pi}</angle_max>
+                <range_min>0.15</range_min>
+                <range_max>12.0</range_max>
+                <noise_stddev>0.003</noise_stddev>
+            </plugin>
         </gazebo>
     </xacro:macro>

File: ros2_ws/description/robot.urdf.xacro (robot description, xacro)
@@ -1,4 +1,19 @@
 <?xml version="1.0"?>
 <robot xmlns:xacro="http://www.ros.org/wiki/xacro" name="robot">
+    <!-- Simulation is the current default.  A real-hardware launch can set
+         use_sim:=false and provide its serial SystemInterface plugin name. -->
+    <xacro:arg name="use_sim" default="true"/>
+    <xacro:arg name="hardware_plugin"
+               default="gz_ros2_control/GazeboSimSystem"/>
+    <xacro:arg name="controllers_file"
+               default="$(find tai_robot_one)/config/ros2_controllers.yaml"/>
+    <!-- Real-hardware parameters are ignored by gz_ros2_control. Stable udev
+         symlinks are mandatory because ttyUSB numbering is not deterministic. -->
+    <xacro:arg name="drive_serial_port" default="/dev/tai_drive"/>
+    <xacro:arg name="lift_serial_port" default="/dev/tai_lift"/>
+    <xacro:arg name="home_lift_on_activate" default="true"/>
+    <xacro:arg name="serial_startup_timeout_ms" default="3000"/>
+    <xacro:arg name="serial_telemetry_timeout_ms" default="250"/>
+    <xacro:arg name="lift_home_timeout_ms" default="70000"/>
     <xacro:include filename="robot_core.xacro"/>
 </robot>

File: ros2_ws/description/robot_core.xacro (robot description, xacro)
@@ -7,4 +7,5 @@
     <xacro:include filename="camera_astra_pro.xacro"/>
     <xacro:include filename="sensor_mount.xacro"/>
+    <xacro:include filename="ros2_control.xacro"/>
     <xacro:include filename="gazebo_control.xacro"/>
     <xacro:include filename="battery_pack.xacro"/>
@@ -19,4 +20,9 @@
     <xacro:property name="wheel_radius" value="0.0875"/>
     <xacro:property name="wheel_width" value="0.035"/>
+    <!-- Safety limit used by both the body controller and each wheel command
+         interface.  0.50 m/s corresponds to 5.714 rad/s at this radius. -->
+    <xacro:property name="max_vehicle_linear_speed" value="0.50"/>
+    <xacro:property name="max_wheel_speed_rad_s"
+                    value="${max_vehicle_linear_speed / wheel_radius}"/>
     <!-- Estimated total mass of one rubber-tyred, plastic-rim wheel. -->
     <xacro:property name="wheel_mass" value="0.5"/>
@@ -386,5 +392,11 @@
     <!-- Rear-mounted 8S2P 32140 LiFePO4 battery inside the chassis. -->
     <xacro:lfp_battery_pack parent="chassis"/>
-    <!-- Native Gazebo Harmonic drive, lift and joint-state systems. -->
-    <xacro:gazebo_control_plugins/>
+    <!-- Stable controller-facing contract shared by simulation and hardware. -->
+    <xacro:tai_robot_ros2_control hardware_plugin="$(arg hardware_plugin)"/>
+    <!-- The Gazebo plugin creates controller_manager inside the simulated
+         model.  A real-hardware launch starts controller_manager itself. -->
+    <xacro:if value="$(arg use_sim)">
+        <xacro:gazebo_ros2_control_plugin
+            controllers_file="$(arg controllers_file)"/>
+    </xacro:if>
 </robot>

Commit message: feat: stabilize real robot localization and navigation

File: ros2_ws/description/camera_astra_pro.xacro (robot description, xacro)
@@ -42,5 +42,5 @@
     </material>
     <xacro:macro name="astra_pro_camera"
-                 params="parent x:=0.0 y:=0.0 z:=0.0">
+                 params="parent x:=0.0 y:=0.0 z:=0.0 pitch:=0.0">
         <!-- camera_link is located at the centre of the forward-facing eye.
              REP-103 axes are X forward, Y left and Z up. -->
@@ -48,5 +48,5 @@
             <parent link="${parent}"/>
             <child link="camera_link"/>
-            <origin xyz="${x} ${y} ${z}" rpy="0 0 0"/>
+            <origin xyz="${x} ${y} ${z}" rpy="0 ${pitch} 0"/>
         </joint>
         <link name="camera_link">

File: ros2_ws/description/lidar.xacro (robot description, xacro)
@@ -17,9 +17,9 @@
     </material>
     <xacro:macro name="fork_mast_lidar"
-                 params="parent x:=0.0 y:=0.0 z:=0.0">
+                 params="parent x:=0.0 y:=0.0 z:=0.0 yaw:=0.0">
         <joint name="lidar_joint" type="fixed">
             <parent link="${parent}"/>
             <child link="lidar_link"/>
-            <origin xyz="${x} ${y} ${z}" rpy="0 0 0"/>
+            <origin xyz="${x} ${y} ${z}" rpy="0 0 ${yaw}"/>
         </joint>
         <!-- lidar_link is the optical scan plane. Its absolute height is set

File: ros2_ws/description/robot_core.xacro (robot description, xacro)
@@ -393,10 +393,13 @@
     </xacro:if>
     <xacro:unless value="$(arg use_sim)">
-        <xacro:mast_sensor_mount parent="mast_frame" include_lidar="false"/>
-        <!-- Chassis front is +0.3005 m. The scan axis is 0.437 m behind that
-             edge, hence x=-0.1365 m. The A1M8 scan plane is 50 mm above its
-             bottom, which rests on the 0.335 m-high chassis top. -->
+        <!-- The camera on the real bracket is pitched 20 degrees downward. -->
+        <xacro:mast_sensor_mount parent="mast_frame" include_lidar="false"
+                                 camera_pitch="${-20.0 * pi / 180.0}"/>
+        <!-- Real-robot scan alignment calibration: the temporary lidar mount
+             is 0.2115 m behind base_footprint. The A1M8 scan plane is 50 mm
+             above its bottom, which rests on the 0.335 m-high chassis top. -->
         <xacro:fork_mast_lidar parent="base_footprint"
-                               x="-0.1365" y="0.0" z="0.385"/>
+                               x="-0.2115" y="0.0" z="0.385"
+                               yaw="${-2.0 * pi / 180.0}"/>
     </xacro:unless>
     <!-- BNO055 mounted near the centre of the chassis top surface. -->

File: ros2_ws/description/ros2_control.xacro (robot description, xacro)
@@ -35,4 +35,8 @@
                 </state_interface>
                 <state_interface name="velocity"/>
+                <xacro:unless value="$(arg use_sim)">
+                    <state_interface name="pid_target_velocity"/>
+                    <state_interface name="pid_output_pwm"/>
+                </xacro:unless>
             </joint>
             <joint name="front_right_wheel_joint">
@@ -45,4 +49,8 @@
                 </state_interface>
                 <state_interface name="velocity"/>
+                <xacro:unless value="$(arg use_sim)">
+                    <state_interface name="pid_target_velocity"/>
+                    <state_interface name="pid_output_pwm"/>
+                </xacro:unless>
             </joint>
             <joint name="rear_left_wheel_joint">
@@ -55,4 +63,8 @@
                 </state_interface>
                 <state_interface name="velocity"/>
+                <xacro:unless value="$(arg use_sim)">
+                    <state_interface name="pid_target_velocity"/>
+                    <state_interface name="pid_output_pwm"/>
+                </xacro:unless>
             </joint>
             <joint name="rear_right_wheel_joint">
@@ -65,4 +77,8 @@
                 </state_interface>
                 <state_interface name="velocity"/>
+                <xacro:unless value="$(arg use_sim)">
+                    <state_interface name="pid_target_velocity"/>
+                    <state_interface name="pid_output_pwm"/>
+                </xacro:unless>
             </joint>
             <!-- Position is metres above the mechanical lower stop. In real

File: ros2_ws/description/sensor_mount.xacro (robot description, xacro)
@@ -49,5 +49,6 @@
         <color rgba="0.85 0.035 0.02 1"/>
     </material>
-    <xacro:macro name="mast_sensor_mount" params="parent include_lidar:=true">
+    <xacro:macro name="mast_sensor_mount"
+                 params="parent include_lidar:=true camera_pitch:=0.0">
         <!-- The mount frame lies on the laser scan plane. Because the mast is
              fixed, lifting the fork carriage does not move either sensor. -->
@@ -112,5 +113,6 @@
                                 x="${camera_x_on_mount}" y="0"
                                 z="${camera_eye_height_ground
-                                     - lidar_scan_height_ground}"/>
+                                     - lidar_scan_height_ground}"
+                                pitch="${camera_pitch}"/>
     </xacro:macro>
 </robot>

Commit message: Stabilize simulated camera and prefer shorter Nav2 routes

File: ros2_ws/description/camera_astra_pro.xacro (robot description, xacro)
@@ -9,9 +9,10 @@
     <xacro:property name="astra_vertical_fov" value="${49.5 * pi / 180.0}"/>
     <xacro:property name="astra_diagonal_fov" value="${73.0 * pi / 180.0}"/>
-    <!-- Laptop-friendly simulation profile. 320 x 240 at 10 Hz preserves the
-         camera geometry while producing 12x fewer pixels per second than
-         640 x 480 at 30 Hz. -->
-    <xacro:property name="astra_image_width" value="320"/>
-    <xacro:property name="astra_image_height" value="240"/>
+    <!-- Keep the simulated depth cloud responsive on the navigation laptop.
+         160 x 120 at 10 Hz preserves the camera FOV and supplies several
+         samples per one-degree obstacle-scan bin while cutting cloud work by
+         four versus the previous 320 x 240 profile. -->
+    <xacro:property name="astra_image_width" value="160"/>
+    <xacro:property name="astra_image_height" value="120"/>
     <xacro:property name="astra_update_rate" value="10"/>
     <xacro:property name="astra_fx"
